Commit message: add new urdf

File: low-level/resources/robots/b2_z1_lidar_mount/urdf/b2_z1_lidar_mount.urdf (robot description, URDF)
Before this commit: robot b2_z1_description, 27 links, 26 joints
Joints:
- joint z1_mount_joint: origin xyz=0.0 0 0.09 rpy=0 0 0 -> xyz=0.34218 0 0.23851 rpy=0 0 0

File: low-level/resources/robots/b2_z1_lidar_mount_fast/urdf/b2_z1_lidar_mount_fast.urdf (robot description, URDF)
Before this commit: robot b2_z1_description, 27 links, 26 joints
Links:
- link FL_hip: geometry visual mesh filename=../assets/FL_hip.obj scale=1 1 1
- link FR_hip: geometry visual mesh filename=../assets/FR_hip.obj scale=1 1 1
- link RL_hip: geometry visual mesh filename=../assets/RL_hip.obj scale=1 1 1
- link RR_hip: geometry visual mesh filename=../assets/RR_hip.obj scale=1 1 1
- link base_link: geometry collision box size=0.50 0.28 0.15; visual mesh filename=../assets/base_link.obj scale=1 1 1
Joints:
- joint z1_mount_joint: origin xyz=0.0 0 0.09 rpy=0 0 0 -> xyz=0.34218 0 0.23851 rpy=0 0 0
