Commit message: fix urdf

File: low-level/resources/robots/b1z1/urdf/b1z1.urdf (robot description, URDF)
Before this commit: robot b1z1_description, 29 links, 28 joints
Joints:
- joint base_static_joint: origin xyz=0.3 0 0.09>> rpy=0 0 0 -> xyz=0.3 0 0.09 rpy=0 0 0

File: low-level/resources/robots/b2_z1_lidar_mount_fast/urdf/b2_z1_lidar_mount_fast.urdf (robot description, URDF)
Before this commit: robot b2_z1_lidar_mount_fast_description, 27 links, 26 joints
Links:
- added link ee_gripper_link, mass 0.001
- link gripperMover: geometry collision mesh filename=../assets/z1_GripperMover_col_1.stl; collision mesh filename=../assets/z1_GripperMover_col_2.stl
- link gripperStator: geometry collision mesh filename=../assets/z1_GripperStator_col_1.stl; collision mesh filename=../assets/z1_GripperStator_col_2.stl
Joints:
- removed joint gripperMover_fixed
- added joint ee_gripper: type fixed, parent gripperStator, child ee_gripper_link, origin xyz=0.135 0 0 rpy=0 0 0
- added joint z1_jointGripper: type revolute, parent gripperStator, child gripperMover, origin xyz=0.049 0 0 rpy=0 0 0, axis 0 1 0, limit lower=-1.5707963267948966 upper=0.0 effort=30.0 velocity=10
