Commit message: second version

File: low-level/resources/robots/b2_z1_lidar_mount_fast/urdf/b2_z1_lidar_mount_fast.urdf (robot description, URDF)
Before this commit: robot b2_z1_lidar_mount_fast_description, 27 links, 26 joints
Links:
- added link base; visual box size=0.001 0.001 0.001
- link gripperMover: geometry collision mesh filename=../../b1z1/meshes/z1_GripperMover.dae scale=1 1 1; visual mesh filename=../../b1z1/meshes/z1_GripperMover.dae scale=1 1 1
- link gripperStator: geometry collision mesh filename=../../b1z1/meshes/z1_GripperStator.dae scale=1 1 1; visual mesh filename=../../b1z1/meshes/z1_GripperStator.dae scale=1 1 1
- link link00: geometry collision cylinder length=0.03 radius=0.0325; visual mesh filename=../../b1z1/meshes/z1_Link00.dae scale=1 1 1
- link link01: geometry visual mesh filename=../../b1z1/meshes/z1_Link01.dae scale=1 1 1
- link link02: geometry collision cylinder length=0.051 radius=0.0325; collision cylinder length=0.102 radius=0.02
- link link03: geometry collision cylinder length=0.059 radius=0.0325; collision cylinder length=0.116 radius=0.02
- link link04: geometry collision cylinder length=0.073 radius=0.0325; visual mesh filename=../../b1z1/meshes/z1_Link04.dae scale=1 1 1
- link link05: geometry visual mesh filename=../../b1z1/meshes/z1_Link05.dae scale=1 1 1
- link link06: geometry collision cylinder length=0.051 radius=0.0325; visual mesh filename=../../b1z1/meshes/z1_Link06.dae scale=1 1 1
Joints:
- removed joint gripperStator_fixed
- added joint floating_base: type fixed, parent base, child base_link, origin xyz=0 0 0 rpy=0 0 0
- added joint z1_gripperStator: type fixed, parent link06, child gripperStator, origin xyz=0.051 0.0 0.0 rpy=0 0 0
- joint ee_gripper: axis (none) -> 1 0 0
- joint z1_elbow: limit lower=-2.8797932657906435 upper=0 effort=30 velocity=3.1415 -> lower=-4.782202150464463 upper=-0.4 effort=30.0 velocity=10
- joint z1_forearm_roll: limit lower=-1.3439035240356338 upper=1.3439035240356338 effort=30 velocity=3.1415 -> lower=-1.7278759594743864 upper=1.7278759594743864 effort=30.0 velocity=10; origin xyz=0.07 0 0 rpy=0 0 0 -> xyz=0.07 0.0 0.0 rpy=0 0 0
- joint z1_jointGripper: origin xyz=0.049 0 0 rpy=0 0 0 -> xyz=0.049 0.0 0 rpy=0 0 0
- joint z1_mount_joint: parent base_link -> base
- joint z1_shoulder: limit lower=0 upper=2.9670597283903604 effort=60 velocity=3.1415 -> lower=0.0 upper=3.141592653589793 effort=60.0 velocity=10
- joint z1_waist: limit lower=-2.6179938779914944 upper=2.6179938779914944 effort=30 velocity=3.1415 -> lower=-2.6179938779914944 upper=2.6179938779914944 effort=30.0 velocity=10
- joint z1_wrist_angle: limit lower=-1.5184364492350666 upper=1.5184364492350666 effort=30 velocity=3.1415 -> lower=-1.7453292519943295 upper=1.5707963267948966 effort=30.0 velocity=10
- joint z1_wrist_rotate: limit lower=-2.792526803190927 upper=2.792526803190927 effort=30 velocity=3.1415 -> lower=-2.792526803190927 upper=2.792526803190927 effort=30.0 velocity=10; origin xyz=0.0492 0 0 rpy=0 0 0 -> xyz=0.0492 0.0 0.0 rpy=0 0 0
